File: LoRa/LoRa.kicad_pcb (KiCad board)
At the start: 4 copper layers, 45.9 x 16.1 mm, 36 parts, among them IC1 SX1281IMLTRT, IC2 LD1085D2T33R, IC3 SKY65383-11, IC4 TPS7A20285PDBVR, J1 Conn_01x02_Socket, J2 Conn_01x02_Socket, J6 Conn_Coaxial, U1 ESP32-PICO-D4, Y2 ECS-TXO-20CSMV4-500-AN-TR

Commit message: update
Parts:
- moved FB1 4.85 mm to (128.6, 71.5)
- moved C23 2.50 mm to (129.9, 71.5)
- moved C24 2.50 mm to (134.4, 71.5)
- moved C25 2.50 mm to (132.9, 71.5)
- moved C26 2.50 mm to (131.4, 71.5)
- moved Y2 1.97 mm to (119.1, 74.9)
- moved J6 0.22 mm to (140.6, 77.3)
- moved FL1 0.17 mm to (136.0, 77.3)
- moved ANT1 0.07 mm to (98.2, 84.5)
Routing:
- net VCC_PA: track 15.6 -> 23.9 mm
- net GND: track 18.8 -> 26.6 mm, vias 65 -> 112
- net TCXO: track 3.77 -> 1.73 mm
- net Net-(Y2-VDD): track 3.18 -> 4.69 mm, vias 0 -> 2
- net SX_SCK: track 24.2 -> 25.3 mm
- net CRX: track 25.9 -> 25.2 mm
- net CTX: track 27.7 -> 28.4 mm
- net SX_MOSI: track 24.7 -> 25.3 mm
- net +3.3V: track 16.3 -> 16.6 mm, vias 20 -> 22
- net +2V85: track 17.1 -> 17.4 mm, vias 1 -> 0
Other:
- outline, holes or cut-outs redrawn
